Commit message: "save"

File: src/curobo/content/assets/robot/franka_description/double_franka.urdf (robot description, URDF)
Before this commit: robot double_franka, 31 links, 30 joints
Joints:
- joint base_fixture_j_base_link: origin xyz=0.75 0.75 0 rpy=0 0 0 -> xyz=0.30 0.75 0 rpy=0 0 0
- joint base_fixture_j_base_link_1: origin xyz=-0.75 0.75 0 rpy=0 0 0.0 -> xyz=-0.30 0.75 0 rpy=0 0 0.0
